File: hardware/dev-board/dev-board.kicad_sch (KiCad schematic)
At the start: 48 parts, among them J102 DISC1-P1, J103 DISC1-P2, J3 Conn_01x02_Pin, U102 CDCE913PW, U103 AMS1117-1.8

Commit message: fix devboard sch
Other:
- note added: "I2C ADDR 0xCA"
- note removed: "I2C ADDR 0x65"
Changed lines of the file:
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@@
     (effects (font (size 1.27 1.27)) (justify left bottom))
   )
-  (text "I2C ADDR 0x65" (at 113.03 194.31 0)
+  (text "I2C ADDR 0xCA" (at 113.03 194.31 0)
     (effects (font (size 1.27 1.27)) (justify left bottom))
   )
